File: MCU_Schematic.kicad_sch (KiCad schematic)
At the start: 15 parts, among them SW1 Button, U2 STM32F205RGTx

Commit message: Added microcontroller, organized
Parts:
- removed C10, C9: 2.2 uF, 10uF_Capacitor_FP_GRM188R61C106MAALD:CAPC1608X95N, symbol 10uF_Capacitor_GRM188R61C106MAALD:GRM188R61C106MAALD
- removed C10, C11, C13, C14, C15, C16: 0.1 uF, 10uF_Capacitor_FP_GRM188R61C106MAALD:CAPC1608X95N, symbol 10uF_Capacitor_GRM188R61C106MAALD:GRM188R61C106MAALD
- removed C12: 10 uF, 10uF_Capacitor_FP_GRM188R61C106MAALD:CAPC1608X95N, symbol 10uF_Capacitor_GRM188R61C106MAALD:GRM188R61C106MAALD
- removed C17: 0.1uF, C0805C104K5RACTU:CAPC2012X88N, symbol Capacitor0.1u_C0805C104K5RACTU:C0805C104K5RACTU
- removed C9: 1 uF, 10uF_Capacitor_FP_GRM188R61C106MAALD:CAPC1608X95N, symbol 10uF_Capacitor_GRM188R61C106MAALD:GRM188R61C106MAALD
- removed R5, R6: 10 kOhm, 51Ohm_Resistor_FP:RES_RK73B_1J_KOA, symbol 51Ohm_Resistor:RK73B1JTTD510J
- removed SW1: Button, Button_FP_FSM4JSMA:TE_FSM4JSMA, symbol Button_FSM4JSMA:FSM4JSMA
- removed U2: STM32F205RGTx, Package_QFP:LQFP-64_10x10mm_P0.5mm, symbol MCU_ST_STM32F2:STM32F205RGTx
Other:
- note removed: "Microcontroller"
- note removed: "Reset Button"
