File: MouseSchematic.kicad_sch (KiCad schematic)
At the start: 66 parts, among them IC1 AZ1117IH-3.3TRG1, J1 Programming Header, J2 Right Header, J3 Left Header, J4 JST1, J5 JST2, Q1 IR Receiver, Q2 IR Receiver, Q3 IR Receiver, Q4 IR Receiver, Q5 MOSFET, Q6 MOSFET, Q7 MOSFET, Q8 MOSFET, SW1 Button, U1 STM32F205RGTx, U2 L293DD

Commit message: Updated all footprints
Parts:
- removed C16: 10 uF, 10uF_Capacitor_FP_GRM188R61C106MAALD:CAPC1608X95N, symbol 10uF_Capacitor_GRM188R61C106MAALD:GRM188R61C106MAALD
- removed D1: LED, symbol Device:LED
- removed J1: Programming Header, symbol Connector_Generic:Conn_01x04
- removed J2: Right Header, symbol Connector:Conn_01x06_Pin
- removed J3: Left Header, symbol Connector:Conn_01x06_Pin
- removed R19: R_US, symbol Device:R_US
- added C26: 10uF, CL21B106KOQNNNE:CAPC2012X140N, symbol Capacitor10u_CL21B106KOQNNNE:CL21B106KOQNNNE
- added D1: LTST-C170GKT, LTST-C170GKT:LED_LTST-C170GKT, symbol LEDGreen_LTST-C170GKT:LTST-C170GKT
- added J1, J2: Right Header, 6130XX11121_61300611121:61300611121, symbol Connector01x06_6130XX11121_61300611121:6130XX11121_61300611121
- added J6: Programming Header, B4B-XH-A:JST_B4B-XH-A, symbol Connector1x4_B4B-XH-A:B4B-XH-A
- added R19: RG2012N-121-W-T1, RG2012N-121-W-T1:RESC2012X50N, symbol Resistor120_RG2012N-121-W-T1:RG2012N-121-W-T1
- added S1: EG1218, EG1218:SW_EG1218, symbol Switch_EG1218:EG1218
- R10, R15, R6, R8: footprint ERA6AEB473V:RES_ERA6AEB473V -> ERA_6AEB473V:RES_ERA6AEB473V
- R11, R12, R13, R14: footprint RC0805FR-0751RL:RESC2012X60N -> RC0805FR_0751RL:RESC2012X60N
- R17, R18: footprint 51Ohm_Resistor_FP:RES_RK73B_1J_KOA -> RC0805JR-0710KL:RESC2012X60N
- SW1: footprint Button_FP_FSM4JSMA:TE_FSM4JSMA -> FSM4JSMA:TE_FSM4JSMA
- renumbered C19 to C10, C23 to C19, C22 to C21, C26 to C22, C21 to C23
Connections:
- net 3V3: now also C26.2, D1.2, J1.4, J2.4
- net GND: now also C26.1, J1.1, J2.1, J6.3, R19.2
- net ML1: now also J2.6
- net ML2: now also J2.5
- net MR1: now also J1.6
- net MR2: now also J1.5
- net NRST: now also U1.7 (NRST)
- net NSRT: now also J6.1
- net PA0: now also U1.14 (PA0), J1.3
- net PA1: now also U1.15 (PA1), J1.2
- net PA13: now also U1.46 (PA13), J6.2
- net PA14: now also U1.49 (PA14), J6.4
- net PA6: now also U1.22 (PA6)
- net PA7: now also U1.23 (PA7)
- net PA8: now also U1.41 (PA8), J2.3
- net PA9: now also U1.42 (PA9), J2.2
- net PB1: now also U1.27 (PB1)
- net PB3: now also U1.55 (PB3)
- net PB6: now also U1.58 (PB6)
- net PB7: now also U1.59 (PB7)
- net PB8: now also U1.61 (PB8)
- net PB9: now also U1.62 (PB9)
- net PC4: now also U1.24 (PC4)
- net PC5: now also U1.25 (PC5)
- net PC9: now also U1.40 (PC9)
- net VCC: now also S1.1; no longer C24.1, IC1.3 (INPUT)
- new net: C24.1, IC1.3 (INPUT), S1.3
- new net: D1.1, R19.1
- no-connect marks 0 -> 34
Other:
- note added: "Regulator and Power Switch"
- note removed: "Power Switch"
- note removed: "Regulator"
- moved on the sheet: C21
